Commit message: Add video rendering for debug; added lidar output for rover1 baselinesx

File: processing/catkin_ws/src/slam/red-rover.urdf (robot description, URDF)
Before this commit: robot red-rover, 5 links, 4 joints
Links:
- added link radar
Joints:
- added joint radar_link_joint: type fixed, parent base_link, child radar, origin xyz=0.006 0 -0.011 rpy=0 0 0
